File: KicadJE_ADSR_Mega32.sch (KiCad schematic (older format))
At the start: 75 parts, among them J102 OUT2, J105 IN1, J106 IN2, J107 CV2, J108 CV1

Commit message: 5VA on Atmega32A
Parts:
- gave numbers to parts that had none: 53

Commit message: Initial footprints and netlist
Parts:
- C205, C206, C212: footprint Capacitor_SMD:C_0805_2012Metric_Pad1.15x1.40mm_HandSolder -> AJ:C_0805_AJ
- D117, D118, D119, D120, D121, D122, D123, D124: footprint Diode_SMD:D_SOD-123 -> AJ:D_SOD-123
- R105, R106, R107, R108, R111, R112, R201, R202, R203, R204, R209, R210, R213, R214, R215, R216, R217, R218, R219, R220, R221, R222, R223, R224, R225, R226, R227, R228, R229: footprint Resistor_SMD:R_0805_2012Metric_Pad1.15x1.40mm_HandSolder -> AJ:R_0805_AJ

Commit message: Footprint upd
Parts:
- J102, J105, J106, J107, J108, J211: footprint AJ-Dropbox-Kicad:PJ301SM -> AJ:PJ301SM
- U201, U202: footprint AJ-Dropbox-Kicad:AJ_SO-8_5.3x6.2mm_P1.27mm -> AJ:AJ_SO-8_5.3x6.2mm_P1.27mm
Changed lines of the file:
@@
 F 0 "J212" H 10467 6146 50  0000 R CNN
 F 1 "OUT2" H 10467 6055 50  0000 R CNN
-F 2 "AJ-Dropbox-Kicad:PJ301SM" H 10700 6075 50  0001 C CNN
+F 2 "AJ:PJ301SM" H 10700 6075 50  0001 C CNN
 F 3 "~" H 10700 6075 50  0001 C CNN
 	1    10700 6075
@@
 F 0 "J202" H 1567 5871 50  0000 R CNN
 F 1 "IN1" H 1567 5780 50  0000 R CNN
-F 2 "AJ-Dropbox-Kicad:PJ301SM" H 1800 5800 50  0001 C CNN
+F 2 "AJ:PJ301SM" H 1800 5800 50  0001 C CNN
 F 3 "~" H 1800 5800 50  0001 C CNN
 	1    1800 5800
@@
 F 0 "J203" H 1567 6271 50  0000 R CNN
 F 1 "IN2" H 1567 6180 50  0000 R CNN
-F 2 "AJ-Dropbox-Kicad:PJ301SM" H 1800 6200 50  0001 C CNN
+F 2 "AJ:PJ301SM" H 1800 6200 50  0001 C CNN
 F 3 "~" H 1800 6200 50  0001 C CNN
 	1    1800 6200
@@
 F 0 "J204" H 1567 6671 50  0000 R CNN
 F 1 "CV1" H 1567 6580 50  0000 R CNN
-F 2 "AJ-Dropbox-Kicad:PJ301SM" H 1800 6600 50  0001 C CNN
+F 2 "AJ:PJ301SM" H 1800 6600 50  0001 C CNN
 F 3 "~" H 1800 6600 50  0001 C CNN
 	1    1800 6600
@@
 F 0 "J205" H 1567 7121 50  0000 R CNN
 F 1 "CV2" H 1567 7030 50  0000 R CNN
-F 2 "AJ-Dropbox-Kicad:PJ301SM" H 1800 7050 50  0001 C CNN
+F 2 "AJ:PJ301SM" H 1800 7050 50  0001 C CNN
 F 3 "~" H 1800 7050 50  0001 C CNN
 	1    1800 7050
@@
 F 0 "U201" H 8325 4925 50  0000 C CNN
 F 1 "TL072" H 8350 4850 50  0000 C CNN
-F 2 "AJ-Dropbox-Kicad:AJ_SO-8_5.3x6.2mm_P1.27mm" H 8425 4900 50  0001 C CNN
+F 2 "AJ:AJ_SO-8_5.3x6.2mm_P1.27mm" H 8425 4900 50  0001 C CNN
 F 3 "http://www.ti.com/lit/ds/symlink/tl071.pdf" H 8425 4900 50  0001 C CNN
 	1    8425 4900
@@
 F 0 "U201" V 10750 1100 50  0000 C CNN
 F 1 "TL072" V 10750 1625 50  0000 C CNN
-F 2 "AJ-Dropbox-Kicad:AJ_SO-8_5.3x6.2mm_P1.27mm" H 10900 1375 50  0001 C CNN
+F 2 "AJ:AJ_SO-8_5.3x6.2mm_P1.27mm" H 10900 1375 50  0001 C CNN
 F 3 "http://www.ti.com/lit/ds/symlink/tl071.pdf" H 10900 1375 50  0001 C CNN
 	3    10900 1375
@@
 F 0 "U202" H 8325 5975 50  0000 C CNN
 F 1 "TL072" H 8350 5900 50  0000 C CNN
-F 2 "AJ-Dropbox-Kicad:AJ_SO-8_5.3x6.2mm_P1.27mm" H 8425 5950 50  0001 C CNN
+F 2 "AJ:AJ_SO-8_5.3x6.2mm_P1.27mm" H 8425 5950 50  0001 C CNN
 F 3 "http://www.ti.com/lit/ds/symlink/tl071.pdf" H 8425 5950 50  0001 C CNN
 	1    8425 5950
@@
 F 0 "J211" H 10467 5646 50  0000 R CNN
 F 1 "OUT1" H 10467 5555 50  0000 R CNN
-F 2 "AJ-Dropbox-Kicad:PJ301SM" H 10700 5575 50  0001 C CNN
+F 2 "AJ:PJ301SM" H 10700 5575 50  0001 C CNN
 F 3 "~" H 10700 5575 50  0001 C CNN
 	1    10700 5575

Commit message: Encoder 2
Parts:
- added C201, C202, C207, C208: 0R, AJ:C_0805_AJ, symbol Device:C
- added C210, C212: 100n, AJ:C_0805_AJ, symbol Device:C
- added C219: 47n, AJ:C_0805_AJ, symbol Device:C
- added R209, R210: OPEN, AJ:R_0805_AJ, symbol Device:R
- added R226, R230, R234: 10k, AJ:R_0805_AJ, symbol Device:R
- added SW202: Rotary_Encoder_Switch, Rotary_Encoder:RotaryEncoder_Alps_EC11E-Switch_Vertical_H20mm, symbol Device:Rotary_Encoder_Switch
- J202: renamed from J207; footprint Connector_PinSocket_2.54mm:PinSocket_1x06_P2.54mm_Vertical -> Connector_PinSocket_2.54mm:PinSocket_1x03_P2.54mm_Vertical; symbol Connector:Conn_01x06_Female -> Connector:Conn_01x03_Female
- P201: footprint Connectors_IDC:IDC-Header_2x08_Pitch2.54mm_Straight -> Connector_IDC:IDC-Header_2x08_P2.54mm_Vertical
- renumbered C202 to C203, C203 to C204, C102 to C205, C101 to C206, C205 to C209, C206 to C211, C207 to C213, C208 to C214, C209 to C215, C210 to C216, C211 to C217, C212 to C218, C213 to C220, C214 to C221, D117 to D201, D118 to D202, D119 to D203, D120 to D204, D121 to D205, D122 to D206, D123 to D207, D124 to D208, J209 to J203, J210 to J204, J211 to J205, J102 to J206, J105 to J207, J106 to J208, J108 to J209, J107 to J210, J206 to J211, J208 to J212, R105 to R205, R107 to R206, R108 to R207, R106 to R208, R209 to R211, R210 to R212, R112 to R213, R111 to R214, R213 to R215, R214 to R216, R215 to R217, R216 to R218, R217 to R219, R218 to R220, R220 to R221, R221 to R222, R222 to R223, R223 to R224, R219 to R225, R225 to R227, R226 to R228, R224 to R229, R227 to R231, R228 to R232, R229 to R233, U202 to U201
Connections:
- net +5V: now also R226.2, R230.1
- net 27_A3: now also C201.2, C219.1, R234.1; no longer J202.6 (Pin_6), R205.2
- net 28_A4: now also C202.2, C212.1, R230.2, SW202.A; no longer J202.5 (Pin_5), R208.2
- net 29_A5: now also C210.1, R226.1, SW202.B; no longer J202.4 (Pin_4)
- net Flow2_32: now also U201.5 (+); no longer U201.3 (+)
- net GND: now also C210.2, C212.2, C219.2, SW202.C, SW202.S2
- net GNDA: now also R209.2, R210.2
- net Out1_32: now also C207.2; no longer R223.1
- net Out2_32: now also C208.2; no longer R224.1
- net at R222.2, R224.2: now also U201.7; no longer U201.1
- net at R218.1, R220.2: now also U201.6 (-); no longer U201.2 (-)
- new net: C201.1, R205.2, R209.1
- new net: C202.1, R208.2, R210.1
- new net: C207.1, R223.1
- new net: C208.1, R224.1
- new net: R234.2, SW202.S1
Other:
- note added: "Encoder Control 1"
- note added: "Encoder Control 2"
- note removed: "Encoder Control"
- moved on the sheet: C203, C204, C209, C211, C218, D201, D202, D203, D204, D205, D206, D207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
