File: KicadJE_OLED_Board.sch (KiCad schematic (older format))
At the start: 70 parts, among them J101 Out1, J102 Out2, J103 In1.1, J104 In1.2, J105 In1.3, J106 In1.4, U101 TL072, U102 TL072

Commit message: Updating Atmega32A subboard
Changed lines of the file:
@@
 $Descr A4 11693 8268
 encoding utf-8
-Sheet 1 1
+Sheet 1 3
 Title "Kicad JE - Util"
 Date "2020-03-17"
@@
 	1    0    0    -1
 $EndComp
+$Sheet
+S 9000 2500 1525 2500
+U 608CA457
+F0 "KicadJE_ADSR_Mega32" 97
+F1 "KicadJE_ADSR_Mega32.sch" 97
+$EndSheet
 $EndSCHEMATC

Commit message: Cleanup MasterSCH
Parts:
- removed C105, C106: 100n, Capacitor_SMD:C_0805_2012Metric_Pad1.15x1.40mm_HandSolder, symbol Device:C
- removed R106, R117: 100k, Resistor_SMD:R_0805_2012Metric_Pad1.15x1.40mm_HandSolder, symbol Device:R
- removed R111, R112, R122, R123: 10k, Resistor_SMD:R_0805_2012Metric_Pad1.15x1.40mm_HandSolder, symbol Device:R
- removed R118, R119, R120, R121, R128, R129: 20k, Resistor_SMD:R_0805_2012Metric_Pad1.15x1.40mm_HandSolder, symbol Device:R
- removed R124, R125, R130, R131: 1k, Resistor_SMD:R_0805_2012Metric_Pad1.15x1.40mm_HandSolder, symbol Device:R
- removed R126, R127: OPEN, Resistor_SMD:R_0805_2012Metric_Pad1.15x1.40mm_HandSolder, symbol Device:R
- removed TP111: Flow1, TestPoint:TestPoint_THTPad_2.0x2.0mm_Drill1.0mm, symbol Connector:TestPoint
- removed TP112: Flow2, TestPoint:TestPoint_THTPad_2.0x2.0mm_Drill1.0mm, symbol Connector:TestPoint
- removed U101, U102: TL072, AJ-Dropbox-Kicad:AJ_SO-8_5.3x6.2mm_P1.27mm, symbol Amplifier_Operational:TL072
Connections:
- net labels removed: Flow1, Flow2, In1, In2, Inv1, Inv2, Out1, Out2
- wire segments 204 -> 122

Commit message: 5VA on Atmega32A
Parts:
- gave numbers to parts that had none: 1
Changed lines of the file:
@@
 CHECK POTS
 $Comp
-L Device:R R?
+L Device:R R106
 U 1 1 5EA9C392
 P 2375 3550
-AR Path="/5EA9C392" Ref="R?"  Part="1"
+AR Path="/5EA9C392" Ref="R106"  Part="1"
 AR Path="/5C8C5FC0/5EA9C392" Ref="R?"  Part="1"
 AR Path="/5CAAE8D3/5EA9C392" Ref="R?"  Part="1"
 AR Path="/5E4B0DD9/5EA9C392" Ref="R?"  Part="1"
 AR Path="/5F49A670/5EA9C392" Ref="R?"  Part="1"
-F 0 "R?" V 2300 3550 50  0000 C CNN
+F 0 "R106" V 2300 3550 50  0000 C CNN
 F 1 "10k" V 2375 3550 50  0000 C CNN
 F 2 "Resistor_SMD:R_0805_2012Metric_Pad1.15x1.40mm_HandSolder" V 2305 3550 50  0001 C CNN
@@
 	1725 1400 2275 1400
 $Comp
-L power:GND #PWR?
+L power:GND #PWR0104
 U 1 1 6074CFAE
 P 2275 1400
-F 0 "#PWR?" H 2275 1150 50  0001 C CNN
+F 0 "#PWR0104" H 2275 1150 50  0001 C CNN
 F 1 "GND" H 2280 1227 50  0000 C CNN
 F 2 "" H 2275 1400 50  0001 C CNN
@@
 $EndComp
 $Comp
-L power:GND #PWR?
+L power:GND #PWR0102
 U 1 1 6074DAF4
 P 2125 4650
-F 0 "#PWR?" H 2125 4400 50  0001 C CNN
+F 0 "#PWR0102" H 2125 4400 50  0001 C CNN
 F 1 "GND" H 2130 4477 50  0000 C CNN
 F 2 "" H 2125 4650 50  0001 C CNN
@@
 	2125 4650 2175 4650
 $Comp
-L power:GND #PWR?
+L power:GND #PWR0101
 U 1 1 6074F388
 P 1550 6200
-F 0 "#PWR?" H 1550 5950 50  0001 C CNN
+F 0 "#PWR0101" H 1550 5950 50  0001 C CNN
 F 1 "GND" H 1555 6027 50  0000 C CNN
 F 2 "" H 1550 6200 50  0001 C CNN
@@
 Connection ~ 1550 6200
 $Comp
-L power:GND #PWR?
+L power:GND #PWR0105
 U 1 1 6076A6B9
 P 2725 2075
-F 0 "#PWR?" H 2725 1825 50  0001 C CNN
+F 0 "#PWR0105" H 2725 1825 50  0001 C CNN
 F 1 "GND" H 2730 1902 50  0000 C CNN
 F 2 "" H 2725 2075 50  0001 C CNN

Commit message: Initial footprints and netlist
Parts:
- C101, C102: footprint Capacitor_SMD:C_1206_3216Metric_Pad1.42x1.75mm_HandSolder -> Capacitor_SMD:C_1206_3216Metric
- C103, C104: footprint Capacitor_SMD:C_0805_2012Metric_Pad1.15x1.40mm_HandSolder -> AJ:C_0805_AJ
- D103: footprint LED_SMD:LED_0805_2012Metric_Pad1.15x1.40mm_HandSolder -> AJ:D_SOD-123
- D104, D105, D106, D107, D108, D109, D110, D111: footprint Diode_SMD:D_SOD-123 -> AJ:D_SOD-123
- R101, R102, R103, R104, R105, R106, R107, R108, R109, R110, R113, R114, R115, R116: footprint Resistor_SMD:R_0805_2012Metric_Pad1.15x1.40mm_HandSolder -> AJ:R_0805_AJ
Changed lines of the file:
@@
 F 0 "R109" V 2300 4025 50  0000 C CNN
 F 1 "10k" V 2375 4025 50  0000 C CNN
-F 2 "Resistor_SMD:R_0805_2012Metric_Pad1.15x1.40mm_HandSolder" V 2305 4025 50  0001 C CNN
+F 2 "AJ:R_0805_AJ" V 2305 4025 50  0001 C CNN
 F 3 "~" H 2375 4025 50  0001 C CNN
 	1    2375 4025
@@
 F 0 "R105" V 2100 6025 50  0000 C CNN
 F 1 "1k" V 2225 6000 50  0000 C CNN
-F 2 "Resistor_SMD:R_0805_2012Metric_Pad1.15x1.40mm_HandSolder" V 2155 6025 50  0001 C CNN
+F 2 "AJ:R_0805_AJ" V 2155 6025 50  0001 C CNN
 F 3 "~" H 2225 6025 50  0001 C CNN
 	1    2225 6025
@@
 F 0 "R104" V 2100 5325 50  0000 C CNN
 F 1 "1k" V 2225 5325 50  0000 C CNN
-F 2 "Resistor_SMD:R_0805_2012Metric_Pad1.15x1.40mm_HandSolder" V 2155 5325 50  0001 C CNN
+F 2 "AJ:R_0805_AJ" V 2155 5325 50  0001 C CNN
 F 3 "~" H 2225 5325 50  0001 C CNN
 	1    2225 5325
@@
 F 0 "D107" H 2675 4475 50  0000 L CNN
 F 1 "1N1007" H 2625 4300 50  0000 L CNN
-F 2 "Diode_SMD:D_SOD-123" H 2800 4375 50  0001 C CNN
+F 2 "AJ:D_SOD-123" H 2800 4375 50  0001 C CNN
 F 3 "~" H 2800 4375 50  0001 C CNN
 	1    2800 4375
@@
 F 0 "D111" H 2725 4525 50  0000 L CNN
 F 1 "1N1007" H 2700 4700 50  0000 L CNN
-F 2 "Diode_SMD:D_SOD-123" H 2825 4625 50  0001 C CNN
+F 2 "AJ:D_SOD-123" H 2825 4625 50  0001 C CNN
 F 3 "~" H 2825 4625 50  0001 C CNN
 	1    2825 4625
@@
 F 0 "C101" H 2325 1300 50  0000 L CNN
 F 1 "1u" H 2425 1100 50  0000 L CNN
-F 2 "Capacitor_SMD:C_1206_3216Metric_Pad1.42x1.75mm_HandSolder" H 2438 1050 50  0001 C CNN
+F 2 "Capacitor_SMD:C_1206_3216Metric" H 2438 1050 50  0001 C CNN
 F 3 "~" H 2400 1200 50  0001 C CNN
 	1    2400 1200
@@
 F 0 "C102" H 2350 1725 50  0000 L CNN
 F 1 "1u" H 2350 1500 50  0000 L CNN
-F 2 "Capacitor_SMD:C_1206_3216Metric_Pad1.42x1.75mm_HandSolder" H 2438 1450 50  0001 C CNN
+F 2 "Capacitor_SMD:C_1206_3216Metric" H 2438 1450 50  0001 C CNN
 F 3 "~" H 2400 1600 50  0001 C CNN
 	1    2400 1600
@@
 F 0 "R101" V 1275 1450 50  0000 C CNN
 F 1 "22k" V 1375 1450 50  0000 C CNN
-F 2 "Resistor_SMD:R_0805_2012Metric_Pad1.15x1.40mm_HandSolder" V 1305 1450 50  0001 C CNN
+F 2 "AJ:R_0805_AJ" V 1305 1450 50  0001 C CNN
 F 3 "~" H 1375 1450 50  0001 C CNN
 	1    1375 1450
@@
 F 0 "C103" H 2500 1300 50  0000 L CNN
 F 1 "100n" H 2500 1100 50  0000 L CNN
-F 2 "Capacitor_SMD:C_0805_2012Metric_Pad1.15x1.40mm_HandSolder" H 2638 1050 50  0001 C CNN
+F 2 "AJ:C_0805_AJ" H 2638 1050 50  0001 C CNN
 F 3 "~" H 2600 1200 50  0001 C CNN
 	1    2600 1200
@@
 F 0 "C104" H 2550 1725 50  0000 L CNN
 F 1 "100n" H 2525 1475 50  0000 L CNN
-F 2 "Capacitor_SMD:C_0805_2012Metric_Pad1.15x1.40mm_HandSolder" H 2638 1450 50  0001 C CNN
+F 2 "AJ:C_0805_AJ" H 2638 1450 50  0001 C CNN
 F 3 "~" H 2600 1600 50  0001 C CNN
 	1    2600 1600
@@
 F 0 "D103" H 1700 1675 50  0000 R CNN
 F 1 "LED" H 1650 1750 50  0000 R CNN
-F 2 "LED_SMD:LED_0805_2012Metric_Pad1.15x1.40mm_HandSolder" H 1550 1600 50  0001 C CNN
+F 2 "AJ:D_SOD-123" H 1550 1600 50  0001 C CNN
 F 3 "~" H 1550 1600 50  0001 C CNN
 	1    1550 1600
@@
 F 0 "R103" V 1875 6275 50  0000 C CNN
 F 1 "OPEN" V 1800 6200 50  0000 C CNN
-F 2 "Resistor_SMD:R_0805_2012Metric_Pad1.15x1.40mm_HandSolder" V 1730 6200 50  0001 C CNN
+F 2 "AJ:R_0805_AJ" V 1730 6200 50  0001 C CNN
 F 3 "~" H 1800 6200 50  0001 C CNN
 	1    1800 6200
@@
 F 0 "R102" V 1875 5575 50  0000 C CNN
 F 1 "OPEN" V 1800 5500 50  0000 C CNN
-F 2 "Resistor_SMD:R_0805_2012Metric_Pad1.15x1.40mm_HandSolder" V 1730 5500 50  0001 C CNN
+F 2 "AJ:R_0805_AJ" V 1730 5500 50  0001 C CNN
 F 3 "~" H 1800 5500 50  0001 C CNN
 	1    1800 5500
@@
 F 0 "D106" H 2675 3950 50  0000 L CNN
 F 1 "1N1007" H 2625 3775 50  0000 L CNN
-F 2 "Diode_SMD:D_SOD-123" H 2800 3850 50  0001 C CNN
+F 2 "AJ:D_SOD-123" H 2800 3850 50  0001 C CNN
 F 3 "~" H 2800 3850 50  0001 C CNN
 	1    2800 3850
@@
 F 0 "D110" H 2725 4000 50  0000 L CNN
 F 1 "1N1007" H 2700 4175 50  0000 L CNN
-F 2 "Diode_SMD:D_SOD-123" H 2825 4100 50  0001 C CNN
+F 2 "AJ:D_SOD-123" H 2825 4100 50  0001 C CNN
 F 3 "~" H 2825 4100 50  0001 C CNN
 	1    2825 4100
@@
 F 0 "R110" V 2300 4550 50  0000 C CNN
 F 1 "10k" V 2375 4550 50  0000 C CNN
-F 2 "Resistor_SMD:R_0805_2012Metric_Pad1.15x1.40mm_HandSolder" V 2305 4550 50  0001 C CNN
+F 2 "AJ:R_0805_AJ" V 2305 4550 50  0001 C CNN
 F 3 "~" H 2375 4550 50  0001 C CNN
 	1    2375 4550
@@
 F 0 "R107" V 2300 2650 50  0000 C CNN
 F 1 "10k" V 2375 2650 50  0000 C CNN
-F 2 "Resistor_SMD:R_0805_2012Metric_Pad1.15x1.40mm_HandSolder" V 2305 2650 50  0001 C CNN
+F 2 "AJ:R_0805_AJ" V 2305 2650 50  0001 C CNN
 F 3 "~" H 2375 2650 50  0001 C CNN
 	1    2375 2650
@@
 F 0 "D104" H 2675 2575 50  0000 L CNN
 F 1 "1N1007" H 2625 2400 50  0000 L CNN
-F 2 "Diode_SMD:D_SOD-123" H 2800 2475 50  0001 C CNN
+F 2 "AJ:D_SOD-123" H 2800 2475 50  0001 C CNN
 F 3 "~" H 2800 2475 50  0001 C CNN
 	1    2800 2475
@@
 F 0 "D108" H 2725 2625 50  0000 L CNN
 F 1 "1N1007" H 2700 2800 50  0000 L CNN
-F 2 "Diode_SMD:D_SOD-123" H 2825 2725 50  0001 C CNN
+F 2 "AJ:D_SOD-123" H 2825 2725 50  0001 C CNN
 F 3 "~" H 2825 2725 50  0001 C CNN
 	1    2825 2725
@@
 F 0 "D105" H 2675 3100 50  0000 L CNN
 F 1 "1N1007" H 2625 2925 50  0000 L CNN
-F 2 "Diode_SMD:D_SOD-123" H 2800 3000 50  0001 C CNN
+F 2 "AJ:D_SOD-123" H 2800 3000 50  0001 C CNN
 F 3 "~" H 2800 3000 50  0001 C CNN
 	1    2800 3000
@@
 F 0 "D109" H 2725 3150 50  0000 L CNN
 F 1 "1N1007" H 2700 3325 50  0000 L CNN
-F 2 "Diode_SMD:D_SOD-123" H 2825 3250 50  0001 C CNN
+F 2 "AJ:D_SOD-123" H 2825 3250 50  0001 C CNN
 F 3 "~" H 2825 3250 50  0001 C CNN
 	1    2825 3250
@@
 F 0 "R108" V 2300 3175 50  0000 C CNN
 F 1 "10k" V 2375 3175 50  0000 C CNN
-F 2 "Resistor_SMD:R_0805_2012Metric_Pad1.15x1.40mm_HandSolder" V 2305 3175 50  0001 C CNN
+F 2 "AJ:R_0805_AJ" V 2305 3175 50  0001 C CNN
 F 3 "~" H 2375 3175 50  0001 C CNN
 	1    2375 3175
@@
 F 0 "R114" V 3100 3175 50  0000 C CNN
 F 1 "10k" V 3175 3175 50  0000 C CNN
-F 2 "Resistor_SMD:R_0805_2012Metric_Pad1.15x1.40mm_HandSolder" V 3105 3175 50  0001 C CNN
+F 2 "AJ:R_0805_AJ" V 3105 3175 50  0001 C CNN
 F 3 "~" H 3175 3175 50  0001 C CNN
 	1    3175 3175
@@
 F 0 "R113" V 3100 2650 50  0000 C CNN
 F 1 "10k" V 3175 2650 50  0000 C CNN
-F 2 "Resistor_SMD:R_0805_2012Metric_Pad1.15x1.40mm_HandSolder" V 3105 2650 50  0001 C CNN
+F 2 "AJ:R_0805_AJ" V 3105 2650 50  0001 C CNN
 F 3 "~" H 3175 2650 50  0001 C CNN
 	1    3175 2650
@@
 F 0 "R115" V 3100 4025 50  0000 C CNN
 F 1 "10k" V 3175 4025 50  0000 C CNN
-F 2 "Resistor_SMD:R_0805_2012Metric_Pad1.15x1.40mm_HandSolder" V 3105 4025 50  0001 C CNN
+F 2 "AJ:R_0805_AJ" V 3105 4025 50  0001 C CNN
 F 3 "~" H 3175 4025 50  0001 C CNN
 	1    3175 4025
@@
 F 0 "R116" V 3100 4550 50  0000 C CNN
 F 1 "10k" V 3175 4550 50  0000 C CNN
-F 2 "Resistor_SMD:R_0805_2012Metric_Pad1.15x1.40mm_HandSolder" V 3105 4550 50  0001 C CNN
+F 2 "AJ:R_0805_AJ" V 3105 4550 50  0001 C CNN
 F 3 "~" H 3175 4550 50  0001 C CNN
 	1    3175 4550
@@
 F 0 "R106" V 2300 3550 50  0000 C CNN
 F 1 "10k" V 2375 3550 50  0000 C CNN
-F 2 "Resistor_SMD:R_0805_2012Metric_Pad1.15x1.40mm_HandSolder" V 2305 3550 50  0001 C CNN
+F 2 "AJ:R_0805_AJ" V 2305 3550 50  0001 C CNN
 F 3 "~" H 2375 3550 50  0001 C CNN
 	1    2375 3550

Commit message: Footprint upd
Parts:
- J101, J102, J103, J104, J105, J106: footprint AJ-Dropbox-Kicad:PJ301SM -> AJ:PJ301SM
Changed lines of the file:
@@
 F 0 "J103" H 1525 2800 50  0000 C CNN
 F 1 "In1.1" H 1575 2700 50  0000 C CNN
-F 2 "AJ-Dropbox-Kicad:PJ301SM" H 1775 2650 50  0001 C CNN
+F 2 "AJ:PJ301SM" H 1775 2650 50  0001 C CNN
 F 3 "~" H 1775 2650 50  0001 C CNN
 	1    1775 2650
@@
 F 0 "J104" H 1525 3375 50  0000 C CNN
 F 1 "In1.2" H 1575 3275 50  0000 C CNN
-F 2 "AJ-Dropbox-Kicad:PJ301SM" H 1775 3175 50  0001 C CNN
+F 2 "AJ:PJ301SM" H 1775 3175 50  0001 C CNN
 F 3 "~" H 1775 3175 50  0001 C CNN
 	1    1775 3175
@@
 F 0 "J101" H 775 5500 50  0000 C CNN
 F 1 "Out1" H 900 5400 50  0000 C CNN
-F 2 "AJ-Dropbox-Kicad:PJ301SM" H 1200 5325 50  0001 C CNN
+F 2 "AJ:PJ301SM" H 1200 5325 50  0001 C CNN
 F 3 "~" H 1200 5325 50  0001 C CNN
 	1    1200 5325
@@
 F 0 "J106" H 1450 4700 50  0000 C CNN
 F 1 "In1.4" H 1525 4600 50  0000 C CNN
-F 2 "AJ-Dropbox-Kicad:PJ301SM" H 1775 4550 50  0001 C CNN
+F 2 "AJ:PJ301SM" H 1775 4550 50  0001 C CNN
 F 3 "~" H 1775 4550 50  0001 C CNN
 	1    1775 4550
@@
 F 0 "J102" H 750 6175 50  0000 C CNN
 F 1 "Out2" H 900 6100 50  0000 C CNN
-F 2 "AJ-Dropbox-Kicad:PJ301SM" H 1200 6025 50  0001 C CNN
+F 2 "AJ:PJ301SM" H 1200 6025 50  0001 C CNN
 F 3 "~" H 1200 6025 50  0001 C CNN
 	1    1200 6025
@@
 F 0 "J105" H 1525 4225 50  0000 C CNN
 F 1 "In1.3" H 1575 4125 50  0000 C CNN
-F 2 "AJ-Dropbox-Kicad:PJ301SM" H 1775 4025 50  0001 C CNN
+F 2 "AJ:PJ301SM" H 1775 4025 50  0001 C CNN
 F 3 "~" H 1775 4025 50  0001 C CNN
 	1    1775 4025

Commit message: Encoder 2
Parts:
- removed C101, C102: 1u, Capacitor_SMD:C_1206_3216Metric, symbol Device:C
- removed C103, C104: 100n, AJ:C_0805_AJ, symbol Device:C
- removed H102, H103, H104, H105: MountingHole_Pad, AJ:MountingHole_Eurorack3, symbol Mechanical:MountingHole_Pad
- removed J101: Out1, AJ:PJ301SM, symbol Connector:AudioJack2_SwitchT
- removed J102: Out2, AJ:PJ301SM, symbol Connector:AudioJack2_SwitchT
- removed J103: In1.1, AJ:PJ301SM, symbol Connector:AudioJack2_SwitchT
- removed J104: In1.2, AJ:PJ301SM, symbol Connector:AudioJack2_SwitchT
- removed J105: In1.3, AJ:PJ301SM, symbol Connector:AudioJack2_SwitchT
- removed J106: In1.4, AJ:PJ301SM, symbol Connector:AudioJack2_SwitchT
- removed R106, R107, R108, R109, R110: 10k, AJ:R_0805_AJ, symbol Device:R
- removed TP101: Tri, AJ:Jack_6m3, symbol Connector:TestPoint
- removed TP102: SQ, AJ:Jack_6m3, symbol Connector:TestPoint
- removed TP103: In1, AJ:Jack_6m3, symbol Connector:TestPoint
- removed TP104: In2, AJ:Jack_6m3, symbol Connector:TestPoint
- removed TP105: In3, AJ:Jack_6m3, symbol Connector:TestPoint
- removed TP106: SS, AJ:Jack_6m3, symbol Connector:TestPoint
- R102, R103: value OPEN -> 10k
- R104, R105: value 1k -> 10k
- renumbered R113 to R106, R114 to R107, R115 to R108, R116 to R109
Connections:
- wire segments 122 -> 55
