File: ATMega32A.sch (KiCad schematic (older format))
At the start: 18 parts

Commit message: Most components placed
Parts:
- J301: renamed from J?; footprint Connector_PinHeader_2.54mm:PinHeader_1x06_P2.54mm_Vertical -> Connector_PinHeader_2.54mm:PinHeader_1x05_P2.54mm_Vertical; symbol Connector_Generic:Conn_01x06 -> Connector_Generic:Conn_01x05
- gave numbers to parts that had none: 17
Connections:
- net GND: no longer J301.6 (Pin_6)
