File: KicadJE_OLED_Mega32.sch (KiCad schematic (older format))
At the start: 93 parts, among them J201 OLED, J202 ADC Input, J203 Out2, J204 Out1, J205 OUT1, J206 OUT2, J207 IN1, J208 IN2, J209 CV1, J210 CV2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

Commit message: Wiring DAC board - initiated
Connections:
- net InNeg: now reaches P201.1 (-12), P201.2 (-12), R228.1
- net InPos: now reaches P201.10 (+12), P201.9 (+12), R227.1
- net In5V: now reaches P201.11 (+5), P201.12 (+5), R231.1
Changed lines of the file:
@@
 	0    1    1    0
 $EndComp
+Text Label 1625 675  0    39   ~ 0
+InPos
+Text Label 1575 1775 0    39   ~ 0
+InNeg
+Text Label 1600 775  0    39   ~ 0
+In5V
 $EndSCHEMATC
