File: KicadJE_OLED_Board_Only.kicad_pcb (KiCad board)
At the start: 2 copper layers, 170.6 x 128 mm, 300 parts, among them J1 LED 1-6, J101 Out1, J102 IN1, J103 OUT1, J104 OutFlt, J105 INFLT, J106 OUTFLT, J107 In1_Flt, J108 InAmp, J201 OLED, J202 ADC Input, J203 Out2, J204 Out1, J205 OUT1, J206 OUT2, J207 IN1, J208 IN2, J209 CV1, J210 CV2, J211 FrontLED, J212 -12V Front, J301 UART, J302 AVR-ISP-6, J401 Out2, J402 Out1, J403 OUT1, J404 OUT2, J405 IN1, J406 IN2, J407 CV1, J408 CV2, J409 -12V Front, J410 OLED, J411 ADC Input, J412 FrontLED, J501 UART, J502 AVR-ISP-6, P1 Doepfer_Power_16pin, P101 Doepfer_Power_10pin, P201 Doepfer_Power_16pin, P401 Doepfer_Power_16pin, SW201 Rotary_Encoder_Switch, SW202 Rotary_Encoder_Switch, SW401 Rotary_Encoder_Switch, SW402 Rotary_Encoder_Switch, U101 TL072, U201 TL072, U202 TL072, U301 ATmega32A-AU, U401 TL072, U402 MCP4822, U501 ATmega32A-AU, Y301 16MHz, Y501 16MHz

Commit message: BoardOnlyPCB+Gerber
Parts:
- removed the C102 at (250.6, 108.8)
- removed the C104 at (260.6, 108.8)
- removed D4, D5, D6, D7, D8, D9: LED, AJ:D_0805_AJ
- removed H102, H103, H104, H105: MountingHole_Pad, AJ:MountingHole_Eurorack3
- removed the H2 at (239.1, 77.8)
- removed H3, H5: OLED, AJ:M2.7_Plated
- removed the H4 at (262.1, 77.8)
- removed J1: LED 1-6, Connector_PinHeader_2.54mm:PinHeader_1x06_P2.54mm_Vertical_SMD_Pin1Right
- removed P1: Doepfer_Power_16pin, Connector_PinHeader_2.54mm:PinHeader_2x08_P2.54mm_Vertical_SMD
- removed R2, R3, R4, R5, R6, R7: 12k, AJ:R_0805_AJ
- removed the TP102 at (240.6, 114.8)
- removed TP103: In1, AJ:Jack_6m3
- removed TP105: In3, AJ:Jack_6m3
- removed TP106: HS, AJ:Jack_6m3
- removed TP107: OFF1, AJ:Pot_6m3_scale1
- removed TP107: FM, AJ:Jack_6m3
- removed TP108: PWM, AJ:Jack_6m3
- removed TP112: Fine, AJ:Pot_6m3_scale1
Routing:
- net -12VA: track 191.8 -> 82.5 mm, vias 4 -> 3
- net Net-(D4-Pad2): track 34.7 -> 0.00 mm, vias 1 -> 0
- net Net-(D5-Pad2): track 32.4 -> 0.00 mm, vias 1 -> 0
- net Net-(D6-Pad2): track 26.9 -> 0.00 mm, vias 1 -> 0
- net Net-(D7-Pad2): track 25.5 -> 0.00 mm, vias 1 -> 0
- net +12VA: track 98.8 -> 73.4 mm
- net GND: track 432.6 -> 409.6 mm
- net Net-(D8-Pad2): track 19.6 -> 0.00 mm, vias 1 -> 0
- net Net-(D9-Pad2): track 18.8 -> 0.00 mm, vias 1 -> 0
- net 25_A1_DAC: track 45.4 -> 37.0 mm, vias 2 -> 1
- net Net-(D4-Pad1): track 6.38 -> 0.00 mm, vias 1 -> 0
- net Net-(D8-Pad1): track 5.09 -> 0.00 mm, vias 1 -> 0
- net Net-(D9-Pad1): track 4.85 -> 0.00 mm, vias 1 -> 0
- net Net-(D6-Pad1): track 4.36 -> 0.00 mm, vias 1 -> 0
- net Net-(D5-Pad1): track 4.34 -> 0.00 mm, vias 1 -> 0
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Other:
- board size 170.6 x 128 mm -> 100 x 100 mm
